File: simple_heart/simple_heart.kicad_pcb (KiCad board)
At the start: 2 copper layers, 46.3 x 43.2 mm, 28 parts, among them U1 4017, U2 LM555xM, U3 4017

Commit message: PCB Finished
Parts:
- added BT1: CR2032, Battery:BatteryHolder_Keystone_103_1x20mm, B.Cu at (146.5, 88.4)
- added R4: 0, Resistor_SMD:R_1206_3216Metric, F.Cu at (150.3, 94.5)
- added R5: 0, Resistor_SMD:R_1206_3216Metric, F.Cu at (140.9, 91.0)
- added R6: 0, Resistor_SMD:R_1206_3216Metric, F.Cu at (131.2, 93.8)
- added R7: 0, Resistor_SMD:R_1206_3216Metric, F.Cu at (153.1, 94.5)
- R3: value 100 -> 330
- moved R3 100.1 mm to (146.5, 114.4), turned to -90 degrees
- moved D7 57.6 mm to (128.3, 83.8)
- moved D3 57.6 mm to (138.3, 79.3)
- moved D4 57.6 mm to (154.6, 79.3)
- moved D6 57.6 mm to (160.7, 80.0)
- moved C1 57.6 mm to (147.7, 95.3)
- moved C2 57.6 mm to (146.9, 92.4)
- moved D17 57.6 mm to (139.9, 107.5)
- moved D18 57.6 mm to (153.1, 107.5)
- moved D19 57.6 mm to (143.7, 111.3)
- moved D20 57.6 mm to (149.3, 111.3)
- moved D8 57.6 mm to (164.5, 83.8)
- moved U2 57.6 mm to (143.5, 97.4)
- moved D5 57.3 mm to (132.5, 79.8)
- moved U3 57.3 mm to (156.6, 87.7)
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Connections:
- D15 pad 2: /LED8 -> Net-(D15-Pad2)
- D20 pad 2: /LED20 -> Net-(D20-Pad2)
- R1 pad 2: +BATT -> Net-(R1-Pad2)
- U1 pad 13: GND -> Net-(U1-Pad13)
- U2 pad 4: +BATT -> Net-(R1-Pad2)
- U2 pad 8: +BATT -> Net-(R1-Pad2)
Routing:
- net Net-(D10-Pad1): track 0.00 -> 120.4 mm
- net GND: track 4.57 -> 77.6 mm, vias 0 -> 3
- net +BATT: track 4.69 -> 34.5 mm, vias 0 -> 2
- net Net-(R1-Pad2): track 0.00 -> 26.6 mm, vias 0 -> 2
- net /LED19: track 0.00 -> 23.2 mm, vias 0 -> 2
- net /LED5: track 0.00 -> 22.8 mm, vias 0 -> 2
- net /F/10: track 7.40 -> 29.4 mm, vias 0 -> 2
- net /LED6: track 0.00 -> 22.0 mm, vias 0 -> 2
- net /LED13: track 0.00 -> 19.8 mm, vias 0 -> 2
- net /LED10: track 3.64 -> 22.5 mm
- net /LED16: track 0.00 -> 17.3 mm
- net /LED18: track 0.00 -> 16.9 mm
- net Net-(D20-Pad2): track 0.00 -> 16.5 mm
- net /LED20: track 0.00 -> 16.3 mm, vias 0 -> 2
- net /LED9: track 0.00 -> 16.0 mm
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- added copper zone on F.Cu, net (none)
- added copper zone on F.Cu, net GND
Other:
- outline, holes or cut-outs redrawn
