File: simple_heart/simple_heart.kicad_sch (KiCad schematic)
At the start: 42 parts

Commit message: Circuit almost finished
Parts:
- removed R? (x19): 330, symbol Device:R_US
- added BT1: CR2032, Battery:BatteryHolder_Keystone_103_1x20mm, symbol Device:Battery_Cell
- added C1: 10nF, Capacitor_SMD:C_0805_2012Metric, symbol Device:C
- added C2: 100nF, Capacitor_SMD:C_0805_2012Metric, symbol Device:C
- added R1: 4.7k, Resistor_SMD:R_0805_2012Metric, symbol Device:R_US
- added R2: 470k, Resistor_SMD:R_0805_2012Metric, symbol Device:R_US
- added R4, R5: 0, Resistor_SMD:R_1206_3216Metric, symbol Device:R_US
- added U2: LM555xM, Package_SO:SOIC-8_3.9x4.9mm_P1.27mm, symbol Timer:LM555xM
- D1, D10, D11, D12, D13, D14, D15, D16, D17, D18, D19, D2, D20, D3, D4, D5, D6, D7, D8, D9: renamed from D?; footprint (none) -> LED_SMD:LED_0805_2012Metric
- R3: renamed from R?; value 330 -> 100; footprint (none) -> Resistor_SMD:R_0805_2012Metric
- U1, U3: renamed from U?; footprint (none) -> Package_SO:SO-16_3.9x9.9mm_P1.27mm
Connections:
- net +BATT: now also BT1.1 (+), R4.2
- net GND: now also R3.1, U1.13 (CKEN), U3.13 (CKEN), U3.15 (Reset), BT1.2 (-), C1.2, C2.2, R5.1, U2.1 (GND); no longer D1.1 (K), D10.1 (K), D11.1 (K), D12.1 (K), D13.1 (K), D14.1 (K), D15.1 (K), D16.1 (K), D17.1 (K), D18.1 (K), D19.1 (K), D2.1 (K), D20.1 (K), D3.1 (K), D4.1 (K), D5.1 (K), D6.1 (K), D7.1 (K), D8.1 (K), D9.1 (K)
- net LED1: now also D1.2 (A)
- net LED10: now also D19.2 (A)
- net LED11: now also D2.2 (A)
- net LED12: now also D4.2 (A)
- net LED13: now also D6.2 (A)
- net LED14: now also D8.2 (A)
- net LED15: now also D10.2 (A)
- net LED16: now also D12.2 (A)
- net LED17: now also D14.2 (A)
- net LED18: now also D16.2 (A)
- net LED19: now also D18.2 (A)
- net LED2: now also D3.2 (A)
- net LED20: now also D20.2 (A); no longer R3.1
- net LED3: now also D5.2 (A)
- net LED4: now also D7.2 (A)
- net LED5: now also D9.2 (A)
- net LED6: now also D11.2 (A)
- net LED7: now also D13.2 (A)
- net LED8: now also D15.2 (A)
- net LED9: now also D17.2 (A)
- net at R3.2: now also D1.1 (K), D10.1 (K), D11.1 (K), D12.1 (K), D13.1 (K), D14.1 (K), D15.1 (K), D16.1 (K), D17.1 (K), D18.1 (K), D19.1 (K), D2.1 (K), D20.1 (K), D3.1 (K), D4.1 (K), D5.1 (K), D6.1 (K), D7.1 (K), D8.1 (K), D9.1 (K); no longer D20.2 (A)
- net F/10: now reaches U3.14 (CLK)
- net F/10: now also U1.12 (Cout)
- net CLK: now reaches U1.14 (CLK)
- net CLK: now also U2.3 (Q)
- net at U1.15 (Reset): now also R5.2
- new net: R1.1, R2.2, U2.7 (DIS)
- new net: R1.2, R4.1, U2.4 (R), U2.8 (VCC)
- new net: C2.1, R2.1, U2.2 (TR), U2.6 (THR)
- new net: C1.1, U2.5 (CV)
- no-connect marks 0 -> 1
Other:
- note added: "Clock source"
- note added: "LED Ring"
- note added: "Left side"
- note added: "Right side"
- title: (none) -> Heart Gift - 4071
- moved on the sheet: D1, D10, D11, D12, D13, D14, D15, D16, D17, D18, D19, D2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

Commit message: Update schematic
Parts:
- added R6, R7: 0, Resistor_SMD:R_1206_3216Metric, symbol Device:R_US
- R3: value 100 -> 330
Connections:
- net GND: now also U1.15 (Reset); no longer U1.13 (CKEN)
- net LED20: now also R7.2; no longer D20.2 (A)
- net LED8: now also R6.2; no longer D15.2 (A)
- net at R5.2: now also U1.13 (CKEN); no longer U1.15 (Reset)
- new net: D15.2 (A), R6.1
- new net: D20.2 (A), R7.1
Other:
- note added: "Battery"
- moved on the sheet: BT1, D1, D10, D11, D12, D13, D14, D15, D16, D17, D18, D19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
