File: mic_preamplifier/mic_preamplifier.kicad_pcb (KiCad board)
At the start: 2 copper layers, 44.8 x 38.5 mm, 16 parts, among them J1 Conn_01x03_Male, J2 Conn_01x02_Male, J3 Conn_01x02, J4 Conn_01x02_Male, J5 Conn_01x02, U1 LM324

Commit message: Mic preamp
Connections:
- RV2 pad 3: /Signal Amplified A -> unconnected-(RV2-Pad3)
Changed lines of the file:
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@@
   (net 12 "Net-(R2-Pad2)")
   (net 13 "Net-(RV1-Pad2)")
+  (net 14 "unconnected-(RV2-Pad3)")
   (footprint "Connector_PinHeader_2.54mm:PinHeader_1x03_P2.54mm_Vertical" (layer "F.Cu")
     (at 116.475 87 90)
     (descr "Through hole straight pin header, 1x03, 2.54mm pitch, single row")
     (tags "Through hole pin header THT 1x03 2.54mm single row")
-    (property "Sheetfile" "File: mic_preamplifier.kicad_sch")
+    (property "Sheetfile" "mic_preamplifier.kicad_sch")
     (property "Sheetname" "")
     (attr through_hole)
@@
     (descr "simple 2-pin terminal block, pitch 5.08mm, revamped version of bornier2")
     (tags "terminal block bornier2")
-    (property "Sheetfile" "File: mic_preamplifier.kicad_sch")
+    (property "Sheetfile" "mic_preamplifier.kicad_sch")
     (property "Sheetname" "")
     (attr through_hole)
@@
     (descr "Potentiometer, vertical, Bourns 3296W, https://www.bourns.com/pdfs/3296.pdf")
     (tags "Potentiometer vertical Bourns 3296W")
-    (property "Sheetfile" "File: mic_preamplifier.kicad_sch")
+    (property "Sheetfile" "mic_preamplifier.kicad_sch")
     (property "Sheetname" "")
     (attr through_hole)
@@
     (descr "C, Disc series, Radial, pin pitch=2.50mm, , diameter*width=3.8*2.6mm^2, Capacitor, http://www.vishay.com/docs/45233/krseries.pdf")
     (tags "C Disc series Radial pin pitch 2.50mm  diameter 3.8mm width 2.6mm Capacitor")
-    (property "Sheetfile" "File: mic_preamplifier.kicad_sch")
+    (property "Sheetfile" "mic_preamplifier.kicad_sch")
     (property "Sheetname" "")
     (attr through_hole)
@@
     (descr "Through hole straight pin header, 1x02, 2.54mm pitch, single row")
     (tags "Through hole pin header THT 1x02 2.54mm single row")
-    (property "Sheetfile" "File: mic_preamplifier.kicad_sch")
+    (property "Sheetfile" "mic_preamplifier.kicad_sch")
     (property "Sheetname" "")
     (attr through_hole)
@@
     (descr "14-lead though-hole mounted DIP package, row spacing 7.62 mm (300 mils), LongPads")
     (tags "THT DIP DIL PDIP 2.54mm 7.62mm 300mil LongPads")
-    (property "Sheetfile" "File: mic_preamplifier.kicad_sch")
+    (property "Sheetfile" "mic_preamplifier.kicad_sch")
     (property "Sheetname" "")
     (attr through_hole)
@@
     (descr "Resistor, Axial_DIN0207 series, Axial, Horizontal, pin pitch=10.16mm, 0.25W = 1/4W, length*diameter=6.3*2.5mm^2, http://cdn-reichelt.de/documents/datenblatt/B400/1_4W%23YAG.pdf")
     (tags "Resistor Axial_DIN0207 series Axial Horizontal pin pitch 10.16mm 0.25W = 1/4W length 6.3mm diameter 2.5mm")
-    (property "Sheetfile" "File: mic_preamplifier.kicad_sch")
+    (property "Sheetfile" "mic_preamplifier.kicad_sch")
     (property "Sheetname" "")
     (attr through_hole)
@@
     (descr "Through hole straight pin header, 1x02, 2.54mm pitch, single row")
     (tags "Through hole pin header THT 1x02 2.54mm single row")
-    (property "Sheetfile" "File: mic_preamplifier.kicad_sch")
+    (property "Sheetfile" "mic_preamplifier.kicad_sch")
     (property "Sheetname" "")
     (attr through_hole)
@@
     (descr "Resistor, Axial_DIN0207 series, Axial, Horizontal, pin pitch=10.16mm, 0.25W = 1/4W, length*diameter=6.3*2.5mm^2, http://cdn-reichelt.de/documents/datenblatt/B400/1_4W%23YAG.pdf")
     (tags "Resistor Axial_DIN0207 series Axial Horizontal pin pitch 10.16mm 0.25W = 1/4W length 6.3mm diameter 2.5mm")
-    (property "Sheetfile" "File: mic_preamplifier.kicad_sch")
+    (property "Sheetfile" "mic_preamplifier.kicad_sch")
     (property "Sheetname" "")
     (attr through_hole)
@@
     (descr "Resistor, Axial_DIN0207 series, Axial, Horizontal, pin pitch=10.16mm, 0.25W = 1/4W, length*diameter=6.3*2.5mm^2, http://cdn-reichelt.de/documents/datenblatt/B400/1_4W%23YAG.pdf")
     (tags "Resistor Axial_DIN0207 series Axial Horizontal pin pitch 10.16mm 0.25W = 1/4W length 6.3mm diameter 2.5mm")
-    (property "Sheetfile" "File: mic_preamplifier.kicad_sch")
+    (property "Sheetfile" "mic_preamplifier.kicad_sch")
     (property "Sheetname" "")
     (attr through_hole)
@@
     (descr "CP, Radial series, Radial, pin pitch=2.00mm, , diameter=4mm, Electrolytic Capacitor")
     (tags "CP Radial series Radial pin pitch 2.00mm  diameter 4mm Electrolytic Capacitor")
-    (property "Sheetfile" "File: mic_preamplifier.kicad_sch")
+    (property "Sheetfile" "mic_preamplifier.kicad_sch")
     (property "Sheetname" "")
     (attr through_hole)
@@
     (descr "simple 2-pin terminal block, pitch 5.08mm, revamped version of bornier2")
     (tags "terminal block bornier2")
-    (property "Sheetfile" "File: mic_preamplifier.kicad_sch")
+    (property "Sheetfile" "mic_preamplifier.kicad_sch")
     (property "Sheetname" "")
     (attr through_hole)
@@
     (descr "CP, Radial series, Radial, pin pitch=2.00mm, , diameter=4mm, Electrolytic Capacitor")
     (tags "CP Radial series Radial pin pitch 2.00mm  diameter 4mm Electrolytic Capacitor")
-    (property "Sheetfile" "File: mic_preamplifier.kicad_sch")
+    (property "Sheetfile" "mic_preamplifier.kicad_sch")
     (property "Sheetname" "")
     (attr through_hole)
@@
     (descr "Potentiometer, vertical, Bourns 3296W, https://www.bourns.com/pdfs/3296.pdf")
     (tags "Potentiometer vertical Bourns 3296W")
-    (property "Sheetfile" "File: mic_preamplifier.kicad_sch")
+    (property "Sheetfile" "mic_preamplifier.kicad_sch")
     (property "Sheetname" "")
     (attr through_hole)
@@
       (net 8 "/Signal Amplified A") (pinfunction "2") (pintype "passive"))
     (pad "3" thru_hole circle (at -5.08 0 180) (size 1.44 1.44) (drill 0.8) (layers *.Cu *.Mask)
-      (net 8 "/Signal Amplified A") (pinfunction "3") (pintype "passive"))
+      (net 14 "unconnected-(RV2-Pad3)") (pinfunction "3") (pintype "passive"))
     (model "${KICAD6_3DMODEL_DIR}/Potentiometer_THT.3dshapes/Potentiometer_Bourns_3296W_Vertical.wrl"
       (offset (xyz 0 0 0))
@@
     (descr "Through hole straight pin header, 1x02, 2.54mm pitch, single row")
     (tags "Through hole pin header THT 1x02 2.54mm single row")
-    (property "Sheetfile" "File: mic_preamplifier.kicad_sch")
+    (property "Sheetfile" "mic_preamplifier.kicad_sch")
     (property "Sheetname" "")
     (attr through_hole)
@@
     (descr "Through hole straight pin header, 1x02, 2.54mm pitch, single row")
     (tags "Through hole pin header THT 1x02 2.54mm single row")
-    (property "Sheetfile" "File: mic_preamplifier.kicad_sch")
-    (property "Sheetname" "")
-    (attr through_hole)
+    (property "Sheetfile" "mic_preamplifier.kicad_sch")
+    (property "Sheetname" "")
+    (attr through_hole)
