File: mic_preamplifier/mic_preamplifier.kicad_sch (KiCad schematic)
At the start: 16 parts, among them J1 Conn_01x03_Male, J2 Conn_01x02_Male, J3 Conn_01x02, J4 Conn_01x02_Male, J5 Conn_01x02, U1 LM324

Commit message: Mic preamp
Connections:
- net Signal Amplified A: no longer RV2.3
Other:
- moved on the sheet: C1, C2, C3, J1, J2, J3, J4, J5, MK1, R1, R2, R3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
