File: pseudo_walkie_talkie/DAC_8.kicad_sch (KiCad schematic)
At the start: 24 parts

Commit message: Lab project IIE-1C2023
Parts:
- removed C5: 47nF, Capacitor_THT:CP_Radial_D5.0mm_P2.00mm, symbol Device:C_Polarized_Small_US
- added C5: 47nF, Capacitor_THT:C_Disc_D3.8mm_W2.6mm_P2.50mm, symbol Device:C_Small
Connections:
- net DAC OUT: now also C5.1
- net GNDA: now also C5.2
Changed lines of the file:
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@@
-    )
-  )
-  (symbol (lib_id "Device:C_Polarized_Small_US") (at 165.1 66.04 0) (unit 1)
-    (in_bom yes) (on_board yes) (dnp no) (fields_autoplaced)
-    (property "Reference" "C5" (at 167.64 64.3382 0)
-      (effects (font (size 1.27 1.27)) (justify left))
-    )
-    (property "Value" "47nF" (at 167.64 66.8782 0)
-      (effects (font (size 1.27 1.27)) (justify left))
-    )
-    (property "Footprint" "Capacitor_THT:CP_Radial_D5.0mm_P2.00mm" (at 165.1 66.04 0)
-      (effects (font (size 1.27 1.27)) hide)
-    )
-    (property "Datasheet" "~" (at 165.1 66.04 0)
-      (effects (font (size 1.27 1.27)) hide)
-    )
-    (pin "1")
-    (pin "2")
-    (instances
-      (project "pseudo_walkie_talkie"
-        (path "/9815d1f2-b58e-4e11-ae6c-807f9f1997ad/d1767ce7-acac-4b41-bf4e-ebbc025006c0"
-          (reference "C5") (unit 1)
-        )
-      )
     )
   )
@@
         )
       )
+    )
+  )
+  (symbol (lib_id "Device:C_Small") (at 165.1 66.04 0) (unit 1)
+    (in_bom yes) (on_board yes) (dnp no) (fields_autoplaced)
+    (property "Reference" "C5" (at 167.64 64.7763 0)
+      (effects (font (size 1.27 1.27)) (justify left))
+    )
+    (property "Value" "47nF" (at 167.64 67.3163 0)
+      (effects (font (size 1.27 1.27)) (justify left))
+    )
+    (property "Footprint" "Capacitor_THT:C_Disc_D3.8mm_W2.6mm_P2.50mm" (at 165.1 66.04 0)
+      (effects (font (size 1.27 1.27)) hide)
+    )
+    (property "Datasheet" "~" (at 165.1 66.04 0)
+      (effects (font (size 1.27 1.27)) hide)
+    )
+    (pin "1")
+    (pin "2")
+    (instances
+      (project "pseudo_walkie_talkie"
+        (path "/9815d1f2-b58e-4e11-ae6c-807f9f1997ad/d1767ce7-acac-4b41-bf4e-ebbc025006c0"
+          (reference "C5") (unit 1)
+        )
+      )
