File: preperf_10x10/preperf_10x10_V0.kicad_pcb (KiCad board)
At the start: 8 copper layers, 100 x 100 mm, 1363 parts, among them J1 Conn_01x02_Pin, J2 Conn_01x01_Pin, J20 Conn_01x01_Pin, J3 Conn_01x01_Pin, J36 Conn_01x01_Pin, J37 Conn_01x01_Pin, J4 Conn_01x02_Pin, J5 Conn_01x01_Pin, J6 Conn_01x02_Pin, Q3 BC548, Q4 BC558, SW1 SW_DIP_x06, SW2 SW_Push, U1 74LS04, U10 74LS73, U11 74LS73, U12 74LS14, U2 LM7805_TO220, U3 74LS08, U4 74LS32, U5 74LS02, U6 74LS386, U7 7400, U8 4511, U9 D168K

Commit message: Added TP2, TP3 and TP4
Parts:
- removed C11: C, Capacitor_THT:C_Disc_D5.0mm_W2.5mm_P2.50mm
- removed JP1, JP2, JP3: Jumper_3_Bridged12, Connector_PinHeader_2.54mm:PinHeader_1x03_P2.54mm_Vertical
- removed R12, R14: R_US, Resistor_THT:R_Axial_DIN0207_L6.3mm_D2.5mm_P2.54mm_Vertical
- removed R13: R_US, Resistor_THT:R_Axial_DIN0207_L6.3mm_D2.5mm_P7.62mm_Horizontal
- removed RN1: R_Network06_US, Resistor_THT:R_Array_SIP7
- removed SW2: SW_Push, Button_Switch_THT:SW_PUSH_6mm_H7.3mm
- removed U10, U11: 74LS73, Package_DIP:DIP-14_W7.62mm_Socket
- removed U12: 74LS14, Package_DIP:DIP-14_W7.62mm_Socket
- removed U8: 4511, Package_DIP:DIP-16_W7.62mm_Socket
- removed U9: D168K, Display_7Segment:D1X8K
- added J10: Conn_01x01_Pin, Connector_PinHeader_2.54mm:PinHeader_1x01_P2.54mm_Vertical, F.Cu at (188.0, 78.7)
- added J11: Conn_01x01_Pin, Connector_PinHeader_2.54mm:PinHeader_1x01_P2.54mm_Vertical, F.Cu at (180.3, 78.7)
- added J12: Conn_01x06_Pin, Connector_PinHeader_2.54mm:PinHeader_1x06_P2.54mm_Vertical, F.Cu at (81.3, 106.7)
- added J13: Conn_01x02_Pin, Connector_PinHeader_2.54mm:PinHeader_1x02_P2.54mm_Vertical, F.Cu at (132.1, 96.5)
- added J14: Conn_01x02_Pin, Connector_PinHeader_2.54mm:PinHeader_1x02_P2.54mm_Vertical, F.Cu at (139.7, 96.5)
- added J15: Conn_01x02_Pin, Connector_PinHeader_2.54mm:PinHeader_1x02_P2.54mm_Vertical, F.Cu at (144.8, 78.7)
- added J16: Conn_01x02_Pin, Connector_PinHeader_2.54mm:PinHeader_1x02_P2.54mm_Vertical, F.Cu at (137.2, 78.7)
- added J17: Conn_01x01_Pin, Connector_PinHeader_2.54mm:PinHeader_1x01_P2.54mm_Vertical, F.Cu at (137.2, 96.5)
- added J18: Conn_01x01_Pin, Connector_PinHeader_2.54mm:PinHeader_1x01_P2.54mm_Vertical, F.Cu at (144.8, 96.5)
- added J19: Conn_01x01_Pin, Connector_PinHeader_2.54mm:PinHeader_1x01_P2.54mm_Vertical, F.Cu at (147.3, 78.7)
- added J21: Conn_01x01_Pin, Connector_PinHeader_2.54mm:PinHeader_1x01_P2.54mm_Vertical, F.Cu at (154.9, 96.5)
- added J22: Conn_01x01_Pin, Connector_PinHeader_2.54mm:PinHeader_1x01_P2.54mm_Vertical, F.Cu at (160.0, 96.5)
- added J23: Conn_01x01_Pin, Connector_PinHeader_2.54mm:PinHeader_1x01_P2.54mm_Vertical, F.Cu at (165.1, 96.5)
- added J24: Conn_01x01_Pin, Connector_PinHeader_2.54mm:PinHeader_1x01_P2.54mm_Vertical, F.Cu at (167.6, 78.7)
- added J25: Conn_01x01_Pin, Connector_PinHeader_2.54mm:PinHeader_1x01_P2.54mm_Vertical, F.Cu at (162.6, 78.7)
- added J26: Conn_01x01_Pin, Connector_PinHeader_2.54mm:PinHeader_1x01_P2.54mm_Vertical, F.Cu at (157.5, 78.7)
- added J27: Conn_01x01_Pin, Connector_PinHeader_2.54mm:PinHeader_1x01_P2.54mm_Vertical, F.Cu at (152.4, 96.5)
- added J28: Conn_01x01_Pin, Connector_PinHeader_2.54mm:PinHeader_1x01_P2.54mm_Vertical, F.Cu at (157.5, 96.5)
- added J29: Conn_01x01_Pin, Connector_PinHeader_2.54mm:PinHeader_1x01_P2.54mm_Vertical, F.Cu at (162.6, 96.5)
- added J30: Conn_01x01_Pin, Connector_PinHeader_2.54mm:PinHeader_1x01_P2.54mm_Vertical, F.Cu at (165.1, 78.7)
- added J31: Conn_01x01_Pin, Connector_PinHeader_2.54mm:PinHeader_1x01_P2.54mm_Vertical, F.Cu at (160.0, 78.7)
- added J32: Conn_01x01_Pin, Connector_PinHeader_2.54mm:PinHeader_1x01_P2.54mm_Vertical, F.Cu at (154.9, 78.7)
- added J33: Conn_01x02_Pin, Connector_PinHeader_2.54mm:PinHeader_1x02_P2.54mm_Vertical, F.Cu at (22.9, 78.7)
- added J34: Conn_01x02_Pin, Connector_PinHeader_2.54mm:PinHeader_1x02_P2.54mm_Vertical, F.Cu at (22.9, 88.9)
- added J35: Conn_01x02_Pin, Connector_PinHeader_2.54mm:PinHeader_1x02_P2.54mm_Vertical, F.Cu at (35.6, 94.0)
- added J38: Conn_01x01_Pin, Connector_PinHeader_2.54mm:PinHeader_1x01_P2.54mm_Vertical, F.Cu at (22.9, 86.4)
- added J39: Conn_01x01_Pin, Connector_PinHeader_2.54mm:PinHeader_1x01_P2.54mm_Vertical, F.Cu at (35.6, 88.9)
- added J40: Conn_01x01_Pin, Connector_PinHeader_2.54mm:PinHeader_1x01_P2.54mm_Vertical, F.Cu at (35.6, 86.4)
- added J41: Conn_01x02_Pin, Connector_PinHeader_2.54mm:PinHeader_1x02_P2.54mm_Vertical, F.Cu at (38.1, 78.7)
- added J42: Conn_01x02_Pin, Connector_PinHeader_2.54mm:PinHeader_1x02_P2.54mm_Vertical, F.Cu at (38.1, 86.4)
- added J43: Conn_01x02_Pin, Connector_PinHeader_2.54mm:PinHeader_1x02_P2.54mm_Vertical, F.Cu at (50.8, 91.4)
- added J44: Conn_01x02_Pin, Connector_PinHeader_2.54mm:PinHeader_1x02_P2.54mm_Vertical, F.Cu at (50.8, 83.8)
- added J45: Conn_01x01_Pin, Connector_PinHeader_2.54mm:PinHeader_1x01_P2.54mm_Vertical, F.Cu at (38.1, 83.8)
- added J46: Conn_01x01_Pin, Connector_PinHeader_2.54mm:PinHeader_1x01_P2.54mm_Vertical, F.Cu at (38.1, 91.4)
- added J47: Conn_01x01_Pin, Connector_PinHeader_2.54mm:PinHeader_1x01_P2.54mm_Vertical, F.Cu at (50.8, 94.0)
- added J48: Conn_01x01_Pin, Connector_PinHeader_2.54mm:PinHeader_1x01_P2.54mm_Vertical, F.Cu at (50.8, 86.4)
- added J49: Conn_01x02_Pin, Connector_PinHeader_2.54mm:PinHeader_1x02_P2.54mm_Vertical, F.Cu at (53.3, 81.3)
- added J50: Conn_01x02_Pin, Connector_PinHeader_2.54mm:PinHeader_1x02_P2.54mm_Vertical, F.Cu at (53.3, 88.9)
- added J51: Conn_01x02_Pin, Connector_PinHeader_2.54mm:PinHeader_1x02_P2.54mm_Vertical, F.Cu at (66.0, 94.0)
- added J52: Conn_01x02_Pin, Connector_PinHeader_2.54mm:PinHeader_1x02_P2.54mm_Vertical, F.Cu at (66.0, 86.4)
- added J53: Conn_01x01_Pin, Connector_PinHeader_2.54mm:PinHeader_1x01_P2.54mm_Vertical, F.Cu at (53.3, 78.7)
- added J54: Conn_01x01_Pin, Connector_PinHeader_2.54mm:PinHeader_1x01_P2.54mm_Vertical, F.Cu at (53.3, 86.4)
- added J55: Conn_01x01_Pin, Connector_PinHeader_2.54mm:PinHeader_1x01_P2.54mm_Vertical, F.Cu at (66.0, 88.9)
- added J56: Conn_01x01_Pin, Connector_PinHeader_2.54mm:PinHeader_1x01_P2.54mm_Vertical, F.Cu at (66.0, 81.3)
- added J7: Conn_01x02_Pin, Connector_PinHeader_2.54mm:PinHeader_1x02_P2.54mm_Vertical, F.Cu at (172.7, 96.5)
- added J8: Conn_01x01_Pin, Connector_PinHeader_2.54mm:PinHeader_1x01_P2.54mm_Vertical, F.Cu at (177.8, 96.5)
- added J9: Conn_01x01_Pin, Connector_PinHeader_2.54mm:PinHeader_1x01_P2.54mm_Vertical, F.Cu at (185.4, 96.5)
- J2, J3, J36, J5: value Conn_01x01_Pin -> Conn_01x02_Pin; footprint Connector_PinHeader_2.54mm:PinHeader_1x01_P2.54mm_Vertical -> Connector_PinHeader_2.54mm:PinHeader_1x02_P2.54mm_Vertical
- R1, R11, R2, R3, R4, R5: footprint Resistor_THT:R_Axial_DIN0207_L6.3mm_D2.5mm_P2.54mm_Vertical -> Resistor_THT:R_Axial_DIN0207_L6.3mm_D2.5mm_P7.62mm_Horizontal
- U1: value 74LS04 -> 74LS08
- U3: value 74LS08 -> 74LS32
- U4: value 74LS32 -> 74LS04
- U5: value 74LS02 -> 74LS386
- U6: value 74LS386 -> 7400
- U7: value 7400 -> 74LS02
- moved J37 170.7 mm to (22.9, 83.8)
- moved U5 163.5 mm to (25.4, 78.7), turned to 0 degrees
- moved J36 157.8 mm to (35.6, 83.8), turned to 180 degrees
- moved C10 154.3 mm to (35.6, 78.7), turned to 90 degrees
- moved U6 153.5 mm to (40.6, 78.7), turned to 0 degrees
- moved C9 125.5 mm to (50.8, 78.7), turned to 90 degrees
- moved U7 124.6 mm to (55.9, 78.7), turned to 0 degrees
- moved C4 118.6 mm to (66.0, 78.7), turned to 90 degrees
- moved R1 74.1 mm to (182.9, 53.3)
- moved R3 74.1 mm to (182.9, 58.4)
- moved R5 74.1 mm to (182.9, 63.5)
- moved R2 74.1 mm to (182.9, 55.9)
- moved R4 74.1 mm to (182.9, 61.0)
- moved R11 59.5 mm to (182.9, 66.0)
- moved J20 52.1 mm to (139.7, 78.7)
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Connections:
- D1 pad 1: /Logic/A -> /Logic/F
- D2 pad 1: /Logic/B -> /Logic/E
- D3 pad 1: /Logic/C -> /Logic/D
- D7 pad 1: /Logic/D -> /Logic/C
- D8 pad 1: /Logic/E -> /Logic/B
- D9 pad 1: /Logic/F -> /Logic/A
- J3 pad 1: Net-(J3-Pin_1) -> /Logic/B
- J5 pad 1: Net-(J5-Pin_1) -> /Logic/C
- R1 pad 1: Net-(U8-Qa) -> /Logic/F
- R1 pad 2: Net-(U9-A) -> GND
- R11 pad 1: Net-(U8-Qf) -> /Logic/A
- R11 pad 2: Net-(U9-F) -> GND
- R2 pad 1: Net-(U8-Qb) -> /Logic/E
- R2 pad 2: Net-(U9-B) -> GND
- R3 pad 1: Net-(U8-Qc) -> /Logic/D
- R3 pad 2: Net-(U9-C) -> GND
- R4 pad 1: Net-(U8-Qd) -> /Logic/C
- R4 pad 2: Net-(U9-D) -> GND
- R5 pad 1: Net-(U8-Qe) -> /Logic/B
- R5 pad 2: Net-(U9-E) -> GND
- U1 pad 1: unconnected-(U1-Pad1) -> Net-(J7-Pin_1)
- U1 pad 10: unconnected-(U1-Pad10) -> /Logic/A
- U1 pad 11: unconnected-(U1-Pad11) -> /Logic/~{A}C
- U1 pad 12: unconnected-(U1-Pad12) -> /Logic/C
- U1 pad 13: unconnected-(U1-Pad13) -> /Logic/~{A}
- U1 pad 2: unconnected-(U1-Pad2) -> Net-(J7-Pin_2)
- U1 pad 3: unconnected-(U1-Pad3) -> Net-(J8-Pin_1)
- U1 pad 4: unconnected-(U1-Pad4) -> Net-(J2-Pin_1)
- U1 pad 5: unconnected-(U1-Pad5) -> Net-(J2-Pin_2)
- U1 pad 6: unconnected-(U1-Pad6) -> Net-(J9-Pin_1)
- U1 pad 8: Net-(U1-Pad8) -> /Logic/AB
- U1 pad 9: /Logic/A -> /Logic/B
- U3 pad 1: /Logic/LATCH_R -> Net-(J13-Pin_1)
- U3 pad 10: /Logic/B -> /Logic/~{A}C
- U3 pad 11: Net-(U3-Pad11) -> Net-(J20-Pin_1)
- U3 pad 12: /Logic/C -> Net-(J16-Pin_1)
- U3 pad 13: Net-(U1-Pad8) -> Net-(J16-Pin_2)
- U3 pad 2: /Logic/CLK_RS -> Net-(J13-Pin_2)
- U3 pad 3: Net-(U3-Pad3) -> Net-(J17-Pin_1)
- U3 pad 4: /Logic/CLK_RS -> Net-(J14-Pin_1)
- U3 pad 5: /Logic/LATCH_S -> Net-(J14-Pin_2)
- U3 pad 6: Net-(U3-Pad6) -> Net-(J18-Pin_1)
- U3 pad 8: Net-(U3-Pad8) -> Net-(J19-Pin_1)
- U3 pad 9: /Logic/A -> /Logic/AB
- U4 pad 1: unconnected-(U4-Pad1) -> Net-(J27-Pin_1)
- U4 pad 10: unconnected-(U4-Pad10) -> Net-(J25-Pin_1)
- U4 pad 11: Net-(J2-Pin_1) -> Net-(J31-Pin_1)
- U4 pad 12: Net-(U3-Pad8) -> Net-(J26-Pin_1)
- U4 pad 13: Net-(U3-Pad11) -> Net-(J32-Pin_1)
- U4 pad 2: unconnected-(U4-Pad2) -> Net-(J21-Pin_1)
- U4 pad 3: unconnected-(U4-Pad3) -> Net-(J28-Pin_1)
- U4 pad 4: unconnected-(U4-Pad4) -> Net-(J22-Pin_1)
- U4 pad 5: unconnected-(U4-Pad5) -> Net-(J29-Pin_1)
- U4 pad 6: unconnected-(U4-Pad6) -> Net-(J23-Pin_1)
- U4 pad 8: unconnected-(U4-Pad8) -> /Logic/~{A}
- U4 pad 9: unconnected-(U4-Pad9) -> /Logic/A
- U5 pad 1: Net-(J37-Pin_1) -> Net-(J33-Pin_1)
- U5 pad 10: Net-(J3-Pin_1) -> Net-(J39-Pin_1)
- U5 pad 11: unconnected-(U5-Pad11) -> Net-(J40-Pin_1)
- U5 pad 12: unconnected-(U5-Pad12) -> Net-(J36-Pin_1)
- U5 pad 13: unconnected-(U5-Pad13) -> Net-(J36-Pin_2)
- U5 pad 2: Net-(J36-Pin_1) -> Net-(J33-Pin_2)
- U5 pad 3: Net-(U3-Pad6) -> Net-(J37-Pin_1)
- U5 pad 4: Net-(J36-Pin_1) -> Net-(J38-Pin_1)
- U5 pad 5: Net-(U3-Pad3) -> Net-(J34-Pin_1)
- U5 pad 6: Net-(J37-Pin_1) -> Net-(J34-Pin_2)
- U5 pad 8: /Logic/D -> Net-(J35-Pin_1)
- U5 pad 9: Net-(J2-Pin_1) -> Net-(J35-Pin_2)
- U6 pad 1: unconnected-(U6-Pad1) -> Net-(J41-Pin_1)
- U6 pad 10: Net-(J5-Pin_1) -> Net-(J43-Pin_2)
- U6 pad 11: unconnected-(U6-Pad11) -> Net-(J48-Pin_1)
- U6 pad 12: unconnected-(U6-Pad12) -> Net-(J44-Pin_1)
- U6 pad 13: unconnected-(U6-Pad13) -> Net-(J44-Pin_2)
- U6 pad 2: unconnected-(U6-Pad2) -> Net-(J41-Pin_2)
- U6 pad 3: unconnected-(U6-Pad3) -> Net-(J45-Pin_1)
- U6 pad 4: unconnected-(U6-Pad4) -> Net-(J42-Pin_1)
- U6 pad 5: unconnected-(U6-Pad5) -> Net-(J42-Pin_2)
- U6 pad 6: unconnected-(U6-Pad6) -> Net-(J46-Pin_1)
- U6 pad 8: Net-(J3-Pin_1) -> Net-(J47-Pin_1)
- U7 pad 10: /Logic/Q3 -> Net-(J55-Pin_1)
- U7 pad 11: unconnected-(U7-Pad11) -> Net-(J52-Pin_1)
- U7 pad 12: unconnected-(U7-Pad12) -> Net-(J52-Pin_2)
- U7 pad 13: unconnected-(U7-Pad13) -> Net-(J56-Pin_1)
- U7 pad 2: Net-(J5-Pin_1) -> Net-(J49-Pin_1)
- U7 pad 3: Net-(J20-Pin_1) -> Net-(J49-Pin_2)
- U7 pad 4: unconnected-(U7-Pad4) -> Net-(J54-Pin_1)
- U7 pad 5: unconnected-(U7-Pad5) -> Net-(J50-Pin_1)
- U7 pad 6: unconnected-(U7-Pad6) -> Net-(J50-Pin_2)
- U7 pad 9: /Logic/Q1 -> Net-(J51-Pin_2)
Routing:
- net +5V: track 475.0 -> 132.0 mm, vias 14 -> 0
- net GND: track 443.7 -> 167.8 mm, vias 8 -> 0
- net Net-(J51-Pin_1): track 109.2 -> 2.54 mm, vias 8 -> 0
- net /Logic/Q1: track 91.4 -> 0.00 mm, vias 2 -> 0
- net /Logic/Q3: track 90.2 -> 0.00 mm, vias 2 -> 0
- net /Logic/LATCH_S: track 71.1 -> 0.00 mm, vias 2 -> 0
- net /Logic/AB: track 0.00 -> 58.4 mm, vias 0 -> 2
- net Net-(U3-Pad8): track 55.9 -> 0.00 mm
- net /Logic/CLK_RS: track 55.9 -> 0.00 mm, vias 2 -> 0
- net Net-(J53-Pin_1): track 55.9 -> 2.54 mm, vias 2 -> 0
- net Net-(U3-Pad6): track 53.3 -> 0.00 mm, vias 1 -> 0
- net /Logic/~{A}C: track 0.00 -> 48.3 mm, vias 0 -> 2
- net /Logic/CLK_BCD: track 45.7 -> 0.00 mm
- net Net-(U3-Pad11): track 45.7 -> 0.00 mm, vias 1 -> 0
- net Net-(U3-Pad3): track 40.6 -> 0.00 mm
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Other:
- copper layers 8 -> 2
