File: preperf_10x10/_autosave-preperf_10x10.kicad_pcb (KiCad board)
At the start: 2 copper layers, 355.3 x 107.6 mm, 1356 parts, among them J1 Conn_01x02_Pin, J2 Conn_01x02_Pin, J3 Conn_01x02_Pin, J4 Conn_01x01_Pin, J5 Conn_01x01_Pin, J6 Conn_01x01_Pin, J7 Conn_01x01_Pin, J8 Conn_01x01_Pin, J9 Conn_01x01_Pin, Q1 BC548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

Commit message: "TP2" and "TP3" digital techniques
Parts:
- moved REF** 151.2 mm to (602.6, 53.3)
- moved REF** 151.2 mm to (602.6, 148.0)
- moved REF** 151.2 mm to (508.0, 53.3)
- moved REF** 151.2 mm to (508.0, 148.0)
- moved D4 2.54 mm to (147.3, 66.0)
- moved D6 2.54 mm to (147.3, 71.1)
- moved D8 2.54 mm to (147.3, 76.2)
Routing:
- net /Logica/E: track 61.0 -> 63.5 mm
- net /Logica/C: track 50.8 -> 53.3 mm
- net /Logica/A: track 12.7 -> 15.2 mm
- net Net-(D8-A): track 7.62 -> 5.08 mm
- net Net-(D6-A): track 7.62 -> 5.08 mm
- net Net-(D4-A): track 7.62 -> 5.08 mm
Other:
- board size 355.3 x 107.6 mm -> 506.4 x 105.1 mm
