File: preperf_10x10/_autosave-bcd_counter.kicad_sch (KiCad schematic)
At the start: 16 parts, among them U11 74LS73, U12 74LS73, U13 74LS08, U14 74LS32, U8 4511, U9 D168K

Commit message: Added BCD Counter UP (FF JK based)  and Power-On-Reset
Parts:
- R15: footprint Resistor_THT:R_Axial_DIN0207_L6.3mm_D2.5mm_P7.62mm_Horizontal -> Resistor_THT:R_Axial_DIN0207_L6.3mm_D2.5mm_P2.54mm_Vertical
Changed lines of the file:
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@@
       (project "preperf_10x10"
         (path "/7bf6ff06-236f-433e-86e9-cc0b656b998f/5e3fd1e9-02f9-4234-9fa8-a673522c8ef2"
-          (reference "#PWR?") (unit 1)
+          (reference "#PWR0102") (unit 1)
         )
       )
@@
       (project "preperf_10x10"
         (path "/7bf6ff06-236f-433e-86e9-cc0b656b998f/5e3fd1e9-02f9-4234-9fa8-a673522c8ef2"
-          (reference "#PWR?") (unit 1)
+          (reference "#PWR0101") (unit 1)
         )
       )
@@
       (effects (font (size 1.27 1.27)))
     )
-    (property "Footprint" "Resistor_THT:R_Axial_DIN0207_L6.3mm_D2.5mm_P7.62mm_Horizontal" (at 51.054 53.594 90)
+    (property "Footprint" "Resistor_THT:R_Axial_DIN0207_L6.3mm_D2.5mm_P2.54mm_Vertical" (at 51.054 53.594 90)
       (effects (font (size 1.27 1.27)) hide)
     )
@@
       (project "preperf_10x10"
         (path "/7bf6ff06-236f-433e-86e9-cc0b656b998f/5e3fd1e9-02f9-4234-9fa8-a673522c8ef2"
-          (reference "#PWR?") (unit 1)
-        )
-      )
+          (reference "#PWR0103") (unit 1)
+        )
+      )
