File: preperf_10x10/logic_tester.kicad_sch (KiCad schematic)
At the start: 9 parts, among them J3 Conn_01x02_Pin, Q1 BC548, Q2 BC558

Commit message: [ADD] Digital Logic Design project (FIUBA): PCB implementation of schmitt triggers, logic functions, counters, state machines, and logic probes
Parts:
- renumbered D2 to D1, D3 to D2, J3 to J2, R2 to R1, R4 to R2, R5 to R3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
